Commit message: Added documentation for ROS2 project

File: 03 Software/01 ROS2/marc/marc_description/src/urdf/parts/diff_drive_base.urdf.xacro (robot description, xacro)
@@ -10,11 +10,11 @@
             <!-- Settings -->
                <always_on>true</always_on>
-               <update_rate>50</update_rate>
+               <update_rate>40</update_rate>
                <left_joint>left_wheel_joint</left_joint>
                <right_joint>right_wheel_joint</right_joint>
                <wheel_separation>${wheel_separation}</wheel_separation>
                <wheel_diameter>${wheel_radius * 2}</wheel_diameter>
-               <!--<wheel_torque>${wheel_torque}</wheel_torque>-->
-               <!--wheel_acceleration>${wheel_accel}</wheel_acceleration-->
+               <!--<wheel_torque>0.17</wheel_torque>-->
+               <!--<wheel_acceleration>5</wheel_acceleration>-->
                <command_topic>cmd_vel</command_topic>
                <!-- Output -->
@@ -51,7 +51,7 @@
             <inertial>
                 <!-- TODO Mass & Inertia -->
-                <mass value="1" />
-                <origin xyz="0 0 0.0" />
-                <inertia ixx="0.01" ixy="0.0" ixz="0.0" iyy="0.01" iyz="0.0" izz="0.5" />
+                <mass value=".25" />
+                <origin xyz="0 0 0" />
+                <inertia ixx="5." ixy="0.01" ixz="0.01" iyy="5." iyz="0.01" izz="5." />
             </inertial>
         </xacro:base>
@@ -63,8 +63,8 @@
             <origin xyz="0 ${-wheel_separation/2} ${wheel_radius}" rpy="0 0 0"/>
         </xacro:wheel>
-        <xacro:castor prefix="front" radius="${ball_radius}" parent_link="base_link">
+        <xacro:castor prefix="front" radius="${ball_radius-0.001}" parent_link="base_link">
             <origin xyz="${ball_separation / 2} 0 ${ball_radius}" rpy="0 0 0"/>
         </xacro:castor>
-        <xacro:castor prefix="back" radius="${ball_radius}" parent_link="base_link">
+        <xacro:castor prefix="back" radius="${ball_radius-0.001}" parent_link="base_link">
             <origin xyz="${-ball_separation / 2} 0 ${ball_radius}" rpy="0 0 0"/>
         </xacro:castor>

File: 03 Software/01 ROS2/marc/marc_description/src/urdf/parts/lidar_layer.urdf.xacro (robot description, xacro)
@@ -27,7 +27,7 @@
             <inertial>
                 <!-- TODO Mass & Inertia -->
-                <mass value="1" />
+                <mass value="0.2" />
                 <origin xyz="0 0 0.0" />
-                <inertia ixx="0.01" ixy="0.0" ixz="0.0" iyy="0.01" iyz="0.0" izz="0.5" />
+                <inertia ixx="0.5" ixy="0.0" ixz="0.0" iyy="0.5" iyz="0.0" izz="0.05" />
             </inertial>
         </xacro:layer>

File: 03 Software/01 ROS2/marc/marc_description/src/urdf/parts/mechanical/ball_castor.urdf.xacro (robot description, xacro)
@@ -7,6 +7,6 @@
                 <!-- TODO Mass & Inertia -->
                 <origin xyz="0 0 0" />
-                <mass value="0.01" />
-                <inertia ixx="0.001" ixy="0.001" ixz="0.001" iyy="0.001" iyz="0.001" izz="0.001" />
+                <mass value="0.1" />
+                <inertia ixx="0.01" ixy="0.001" ixz="0.001" iyy="0.01" iyz="0.001" izz="0.01" />
             </inertial>
             <visual>
@@ -28,8 +28,12 @@
             <parent link="${parent_link}" />
             <child link="${prefix}_castor_link" />
+            <dynamics damping="0"/>
         </joint>
         <gazebo reference="${prefix}_castor_link">
-           <mu1>0.01</mu1>
-           <mu2>0.01</mu2>
+            <mu1>0.001</mu1>
+            <mu2>0.001</mu2>
+            <!--<kp>100000.0</kp>-->
+            <!--<kd>1000.0</kd>-->
+            <!--<minDepth>0.001</minDepth>-->
         </gazebo>
     </xacro:macro>

File: 03 Software/01 ROS2/marc/marc_description/src/urdf/parts/mechanical/wheel.urdf.xacro (robot description, xacro)
@@ -7,20 +7,20 @@
                 <origin xyz="0 0 0" />
                 <mass value="0.01" />
-            <inertia ixx="0.001" ixy="0.001" ixz="0.001" iyy="0.001" iyz="0.001" izz="0.001" />
-        </inertial>
-        <visual>
-            <origin xyz="0 0 0" rpy="0 ${PI/2} ${PI/2}" />
-            <geometry>
-                <cylinder radius="${radius}" length="${width}" />
-                <material name="red"/>
-            </geometry>
-        </visual>
-        <collision>
-            <origin xyz="0 0 0" rpy="0 ${PI/2} ${PI/2}" />
-            <geometry>
-                <cylinder radius="${radius}" length="${width}" />
-            </geometry>
-            </collision>
-        </link>
+                <inertia ixx="0.01" ixy="0.001" ixz="0.001" iyy="0.01" iyz="0.001" izz="0.01" />
+            </inertial>
+            <visual>
+                <origin xyz="0 0 0" rpy="0 ${PI/2} ${PI/2}" />
+                <geometry>
+                    <cylinder radius="${radius}" length="${width}" />
+                    <material name="red"/>
+                </geometry>
+            </visual>
+            <collision>
+                <origin xyz="0 0 0" rpy="0 ${PI/2} ${PI/2}" />
+                <geometry>
+                    <cylinder radius="${radius}" length="${width}" />
+                </geometry>
+                </collision>
+            </link>
         <joint name="${prefix}_wheel_joint" type="continuous">
             <xacro:insert_block name="origin" />
@@ -28,5 +28,13 @@
             <child link="${prefix}_wheel_link" />
             <axis xyz="0 1 0" />
+            <dynamics damping="0"/>
         </joint>
+        <gazebo reference="${prefix}_wheel_link">
+            <mu1>1.0</mu1>
+            <mu2>1.0</mu2>
+            <kp>100000.0</kp>
+            <kd>1000.0</kd>
+            <!--<minDepth>0.001</minDepth>-->
+        </gazebo>
     </xacro:macro>
 </robot>

File: 03 Software/01 ROS2/marc/marc_description/src/urdf/parts/raspberry_layer.urdf.xacro (robot description, xacro)
@@ -27,7 +27,7 @@
             <inertial>
                 <!-- TODO Mass & Inertia -->
-                <mass value="1" />
+                <mass value="0.2" />
                 <origin xyz="0 0 0.0" />
-                <inertia ixx="0.01" ixy="0.0" ixz="0.0" iyy="0.01" iyz="0.0" izz="0.5" />
+                <inertia ixx="0.3" ixy="0.0" ixz="0.0" iyy="0.3" iyz="0.0" izz="0.05" />
             </inertial>
         </xacro:layer>

File: 03 Software/01 ROS2/marc/marc_description/src/urdf/parts/sensors/CamsenseX1.urdf.xacro (robot description, xacro)
@@ -18,5 +18,42 @@
         </joint>
         <!-- Simulation plugin-->
-         <gazebo reference="lidar_sensor_link">
+        <gazebo reference="lidar_sensor_link">
+            <sensor type="ray" name="CamsenseX1">
+                <ray>
+                    <scan>
+                        <horizontal>
+                            <samples>400</samples>
+                            <resolution>1</resolution>
+                            <min_angle>0</min_angle>
+                            <max_angle>6.283000</max_angle>
+                        </horizontal>
+                        <vertical>
+                            <samples>1</samples>
+                            <resolution>1</resolution>
+                            <min_angle>-0.523</min_angle>
+                            <max_angle>0.523</max_angle>
+                         </vertical>
+                    </scan>
+                    <range>
+                        <min>0.08</min>
+                        <max>8.0</max>
+                        <resolution>0.01</resolution>
+                    </range>
+                    <noise>
+                        <type>gaussian</type>
+                        <mean>0.0</mean>
+                        <stddev>0.01</stddev>
+                    </noise>
+                </ray>
+                <update_rate>5</update_rate>
+                <plugin name="CamsenseX1_plugin" filename="libgazebo_ros_ray_sensor.so">
+                <ros>
+                    <!--<namespace>/lidar</namespace>-->
+                    <remapping>~/out:=scan</remapping>
+                </ros>
+                <output_type>sensor_msgs/LaserScan</output_type>
+                <min_intensity>100.0</min_intensity>
+                </plugin>
+            </sensor>
         </gazebo>
     </xacro:macro>

File: 03 Software/01 ROS2/marc/marc_description/src/urdf/parts/sensors/HC-SR04.urdf.xacro (robot description, xacro)
@@ -44,7 +44,7 @@
                     <ros>
                         <namespace>ultrasonic</namespace>
-                        <remapping>~/out:=ultrasonic/range</remapping>
+                        <remapping>~/out:=range</remapping>
                         <qos>
-                            <topic name="ultrasonic/range">
+                            <topic name="/range">
                                 <publisher>
                                     <reliability>reliable</reliability>

File: 03 Software/01 ROS2/marc/marc_description/src/urdf/parts/sensors/LSM6DS33.urdf.xacro (robot description, xacro)
@@ -19,4 +19,69 @@
         <!-- Simulation plugin-->
         <gazebo reference="${name}_IMU_link">
+            <sensor name="{name}_IMU" type="imu">
+                <plugin filename="libgazebo_ros_imu_sensor.so" name="imu_plugin">
+                    <ros>
+                        <remapping>~/out:=imu</remapping>
+                    </ros>
+                    <initial_orientation_as_reference>false</initial_orientation_as_reference>
+                </plugin>
+                <always_on>true</always_on>
+                <update_rate>50</update_rate>
+                <visualize>true</visualize>
+                <imu>
+                    <angular_velocity>
+                        <x>
+                            <noise type="gaussian">
+                                <mean>0.0</mean>
+                                <stddev>2e-4</stddev>
+                                <bias_mean>0.0000075</bias_mean>
+                                <bias_stddev>0.0000008</bias_stddev>
+                            </noise>
+                        </x>
+                        <y>
+                            <noise type="gaussian">
+                                <mean>0.0</mean>
+                                <stddev>2e-4</stddev>
+                                <bias_mean>0.0000075</bias_mean>
+                                <bias_stddev>0.0000008</bias_stddev>
+                            </noise>
+                        </y>
+                        <z>
+                            <noise type="gaussian">
+                                <mean>0.0</mean>
+                                <stddev>2e-4</stddev>
+                                <bias_mean>0.0000075</bias_mean>
+                                <bias_stddev>0.0000008</bias_stddev>
+                            </noise>
+                        </z>
+                    </angular_velocity>
+                    <linear_acceleration>
+                        <x>
+                            <noise type="gaussian">
+                                <mean>0.0</mean>
+                                <stddev>1.7e-2</stddev>
+                                <bias_mean>0.1</bias_mean>
+                                <bias_stddev>0.001</bias_stddev>
+                            </noise>
+                        </x>
+                        <y>
+                            <noise type="gaussian">
+                                <mean>0.0</mean>
+                                <stddev>1.7e-2</stddev>
+                                <bias_mean>0.1</bias_mean>
+                                <bias_stddev>0.001</bias_stddev>
+                            </noise>
+                        </y>
+                        <z>
+                            <noise type="gaussian">
+                                <mean>0.0</mean>
+                                <stddev>1.7e-2</stddev>
+                                <bias_mean>0.1</bias_mean>
+                                <bias_stddev>0.001</bias_stddev>
+                            </noise>
+                        </z>
+                    </linear_acceleration>
+                </imu>
+            </sensor>
         </gazebo>
     </xacro:macro>

File: 03 Software/01 ROS2/marc/marc_description/src/urdf/parts/sensors/RP_5MP_cam.urdf.xacro (robot description, xacro)
@@ -18,5 +18,59 @@
         </joint>
         <!-- Simulation plugin-->
-         <gazebo reference="${name}_camera_link">
+        <gazebo reference="${name}_camera_link">
+            <sensor type="camera" name="${name}_camera">
+                <always_on>1</always_on>
+                <update_rate>10</update_rate>
+                <visualize>0</visualize>
+                <camera name="${name}_camera">
+                    <horzontal_fov> </horzontal_fov>
+                    <image>
+                        <width>640</width>
+                        <height>480</height>
+                    </image>
+                    <clip>
+                        <near>0.01</near>
+                        <far>100</far>
+                    </clip>
+                    <noise>
+                        <type>gaussian</type>
+                        <mean>0.0</mean>
+                        <stddev>0.1</stddev>
+                    </noise>
+                    <distortion>
+                        <k1>0.</k1>
+                        <k2>0.</k2>
+                        <k3>0.</k3>
+                        <p1>0.</p1>
+                        <p2>0.</p2>
+                        <center>0.5 0.5</center>
+                    </distortion>
+                </camera>
+                <!-- Use camera, not camera_triggered -->
+                <plugin name="RP_5MP_cam" filename="libgazebo_ros_camera.so">
+                    <camera_name>${name}_camera</camera_name>
+                    <frame_name>${name}_camera_optical_frame</frame_name>
+                    <hack_baseline>0.01</hack_baseline>
+                    <ros>
+                        <!-- <namespace>${name}_camera</namespace> -->
+                        <remapping>${name}_camera/image_raw:=color/image_raw</remapping>
+                        <remapping>${name}_camera/camera_info:=color/camera_info</remapping>
+                        <qos>
+                            <topic name="/${name}_camera/color/image_raw">
+                                <publisher>
+                                    <reliability>reliable</reliability>
+                                </publisher>
+                            </topic>
+                        </qos>
+                        <qos>
+                            <topic name="/${name}_camera/color/camera_info">
+                                <publisher>
+                                    <reliability>reliable</reliability>
+                                </publisher>
+                            </topic>
+                        </qos>
+                    </ros>
+                </plugin>
+            </sensor>
         </gazebo>
     </xacro:macro>
